File: RoverControlBoard/RoverControlBoard.sch (KiCad schematic (older format))
At the start: 9 parts

Commit message: finished baord layout
Parts:
- removed P? (x2): CONN_01X03, symbol CONN_01X03
- added P10, P11, P9: CONN_01X02, Pin_Headers:Pin_Header_Straight_1x02_Pitch2.54mm, symbol CONN_01X02
- added P12: CONN_01X03, Pin_Headers:Pin_Header_Straight_1x03_Pitch2.54mm, symbol CONN_01X03
- added Q1: Q_NMOS_GDS, Diodes_ThroughHole:Diode_TO-247_Dual_CommonCathode_Vertical, symbol Q_NMOS_GDS
- added Q2, Q3: Q_NMOS_GDS, Diodes_ThroughHole:Diode_TO-220_Dual_CommonCathode_Vertical, symbol Q_NMOS_GDS
- added R1, R2, R3: R, Resistors_ThroughHole:Resistor_Horizontal_RM7mm, symbol R
- P1, P2, P4, P5: renamed from P?; footprint (none) -> Pin_Headers:Pin_Header_Straight_1x03_Pitch2.54mm
- P7: renamed from P?; footprint (none) -> Pin_Headers:Pin_Header_Straight_1x05_Pitch2.54mm
- SW1: renamed from SW?; footprint (none) -> Buttons_Switches_ThroughHole:SW_DIP_x4_W7.62mm_Slide
- U1: renamed from U?; footprint (none) -> Teensy:Teensy30_31_32_LC
Connections:
- net labels added: D0, D2, D8
- net labels removed: PWMCHAN5, Steering
- wire segments 48 -> 59
- no-connect marks 0 -> 18
Other:
- moved on the sheet: P1, P2, P4, P5, P7, SW1, U1
