File: RoverControlBoard/CtlBoard_V2/ControlBoard.sch (EAGLE design)
At the start: 45 parts, among them U1 PAM8302AASCR, U2 SGTL5000-32

Commit message: added project atomic part library. Finished audio circuit and power switching cirucit, as well as hooked up SD card.
Parts:
- added C13, C14, C17: 2.2uF, ControlBoard:CAP_CERAMIC0805-NOOUTLINE
- added C15, C16, C18: .1uF, ControlBoard:CAP_CERAMIC0805-NOOUTLINE
- added D1, D2: 1A/23V/620mV, SparkFun-DiscreteSemi:DIODE-SCHOTTKY-BAT20J
- added FERRITE_600: (no value), ControlBoard:FERRITE0805
- added JP11, JP12: (no value), pinhead:PINHD-1X3/90
- added Q4: 4.3A/20V/54mΩ, SparkFun-DiscreteSemi:MOSFET_PCH-IRLML2244
- added R8: 10k, resistor:R-US_0207/7
- added VR2: 1V5, ControlBoard:AP7313SOT
- C3: value 10uF -> 1uF
- JP8: device pinhead:PINHD-1X2 -> pinhead:PINHD-1X3/90
- U2: device Freescale:SGTL5000-32 -> ControlBoard:SGTL5000-32
Connections:
- removed net 5V: JP1.2, JP2.2, JP3.2, JP4.2
- removed net AIN-: C2.2, VR1.A
- removed net CS_W25Q: U$1.6/PWM
- removed net SD_?: U$1.14/A0
- removed net SD_?2: U$1.7/RX3
- removed net SD_?3: U$1.10/TX2/PWM
- new net 3V3: C14.2, C15.2, C16.2, FERRITE_600.P$1, U$1.3.3V, U$6.VDD, U2.VDDIO, VR2.VIN
- new net N$29: C17.2, C18.2, FERRITE_600.P$2, U2.VDDA
- new net N$30: C13.2, U2.VDDD, VR2.VOUT
- new net N$31: D2.A, Q4.D
- new net N$33: C8.1, JP11.2
- new net N$35: C9.1, JP12.3
- new net N$36: C10.1, JP12.2
- new net SD_CS: U$1.10/TX2/PWM, U$6.CS
- new net SD_MOSI: U$1.7/RX3, U$6.DATA_IN
- new net SD_SCK: U$1.14/A0, U$6.SCLK
- new net STEERING: JP8.1, U$1.6/PWM
- new net VIN: Q4.S
- new net VUSB: D1.A, Q4.G, R8.2, U$1.VUSB
- new net V_ESC: JP1.2, JP2.2, JP3.2, JP4.2, JP8.2
- net AIN+: now also C7.1, JP11.3
- net GND: now also C13.1, C14.1, C15.1, C16.1, C17.1, C18.1, C2.2, JP11.1, JP12.1, JP8.3, R8.1, U$6.GND, U$6.GND1, U$6.VSS, VR1.A, VR2.GND
- net SD_MISO: now also U$6.DATA_OUT
- net VCC: now also D1.C, D2.C
- net VO+: now also JP9.1
- net VO-: now also JP9.2
Other:
- moved on the sheet: C1, C10, C11, C12, C2, C3, C4, C5, C6, C7, C8, C9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
